File: hw/ewal.brd (EAGLE design)
At the start: 50 x 40 mm, 26 parts, among them U1 MMA8653FC, U2 ATTINY48

Commit message: update to version 2
now with a touch sensor and a different stencil layout for the sensor
Parts:
- added C7: 33n, rcl:C0603
- added R11: 10k, rcl:R0603
Connections:
- new net TOUCH: R11.2
- new net TOUCH1: C7.1, R11.1, U2.8
- new net TOUCH2: C7.2, U2.7
Routing:
- net TOUCH: track 0.00 -> 24.6 mm
- net TOUCH1: track 0.00 -> 4.88 mm
- net VCC: track 113.2 -> 115.9 mm
- net TOUCH2: track 0.00 -> 2.40 mm
- net U: track 19.0 -> 17.5 mm
- net GND: track 17.1 -> 16.4 mm, vias 8 -> 10
- added copper zone on layer 1, net TOUCH
Other:
- board text added: "EWaL2"
- board text removed: "EWaL"
